File: design/hardware/SenSil_v1/SenSil_v1.kicad_sch (KiCad schematic)
At the start: 9 parts, among them J1 RS495, J2 UART, U1 ATmega328P-A, U3 MAX485E

Commit message: Added author and metadata to schematic
Other:
- title: (none) -> Sense Silica
Changed lines of the file:
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@@
 	(generator_version "9.0")
 	(paper "A4")
+	(title_block
+		(title "Sense Silica")
+		(date "2026-01-26")
+		(rev "V1.0")
+		(comment 4 "Author: VigneshRR")
+	)
 	(junction
 		(at 95.25 52.07)
